Commit message: change the mass and inertia of ugv

File: my_ugv/ugv_description/urdf/ugv_robot.urdf.xacro (robot description, xacro)
@@ -22,9 +22,9 @@
     <link name="ugv_base_link">
         <inertial>
-            <mass value="25.0" />
+            <mass value="10.0" />
             <origin xyz="0.0 0.0 0.0" rpy="0 0 0" />
-            <inertia ixx="0.005" ixy="0.0" ixz="0.0"
-                        iyy="0.005" iyz="0.0"
-                        izz="0.005" />
+            <inertia ixx="0.13" ixy="0.0" ixz="0.0"
+                        iyy="0.13" iyz="0.0"
+                        izz="0.13" />
         </inertial>
         <visual>
@@ -49,7 +49,7 @@
             <mass value="0.5" />
             <origin xyz="0.00 0.00 0.1" rpy="0 1.5708 0" />
-            <inertia ixx="0.005" ixy="0.0" ixz="0.0"
-                        iyy="0.005" iyz="0.0"
-                        izz="0.005" />
+            <inertia ixx="0.08" ixy="0.0" ixz="0.0"
+                        iyy="0.08" iyz="0.0"
+                        izz="0.08" />
         </inertial>
         <visual>
@@ -104,5 +104,5 @@
         <plugin name="p3d_base_controller" filename="libgazebo_ros_p3d.so">
             <alwaysOn>true</alwaysOn>
-            <updateRate>50.0</updateRate>
+            <updateRate>30.0</updateRate>
             <bodyName>ugv_base_link</bodyName>
             <topicName>ugv_ground_truth/state</topicName>

Commit message: add embedded apriltag

File: my_ugv/ugv_description/urdf/ugv_robot.urdf.xacro (robot description, xacro)
@@ -57,5 +57,6 @@
             <geometry>
                 <!--<box size="${base_size_x} ${base_size_y} ${base_size_z}" />-->
-                <mesh filename="package://ugv_description/meshes/apriltag/apriltag.dae" scale="1 1 1"/>
+                <!-- <mesh filename="package://ugv_description/meshes/apriltag/apriltag.dae" scale="1 1 1"/> -->
+                <mesh filename="package://ugv_description/meshes/emb_apriltag/emb_apriltag.dae" scale="1 1 1"/>
             </geometry>
         </visual>

Commit message: update car model

File: my_ugv/ugv_description/urdf/ugv_robot.urdf.xacro (robot description, xacro)
@@ -6,31 +6,36 @@
     <!-- Properties (Constants) -->
     <xacro:property name="M_PI" value="3.14159"/>
-    <xacro:property name="base_size_x" value="0.380" />
-    <xacro:property name="base_size_y" value="0.12" />
-    <xacro:property name="base_size_z" value="0.085" />
-    <xacro:property name="wheel_radius_big" value="0.085" />
-    <xacro:property name="wheel_length" value="0.02" />
-    <xacro:property name="wheel_size_y" value="0.0825" />
-    <xacro:property name="total_width" value="0.297" />
+    <xacro:property name="base_size_x" value="2.5" />
+    <xacro:property name="base_size_y" value="1" />
+    <xacro:property name="base_size_z" value="1.2" />
+    <xacro:property name="wheel_radius" value="0.26" />
+    <xacro:property name="wheel_length" value="0.18" />
+    <!-- <xacro:property name="wheel_size_y" value="0.0825" /> -->
     <!--    <xacro:property name="wheel_offset_y" value="${(total_width - wheel_size_y) / 2}" />-->
-    <xacro:property name="wheel_offset_y" value="0.1697" />
-    <xacro:property name="wheel_offset_z_from_base_link" value="-0.0" />
+    <xacro:property name="wheel_offset_y" value="0.48" />
+    <xacro:property name="wheel_offset_z_from_base_link" value="-0.53" />
     <xacro:property name="ground_clearance" value="0.05" />
-    <xacro:property name="top_size_x" value="0.3937" />
-    <xacro:property name="top_size_y" value="0.3556" />
-    <xacro:property name="top_size_z" value="0.0020" />
     <link name="ugv_base_link">
-        <inertial>
-            <mass value="10.0" />
+        <!-- <inertial>
+            <mass value="20.0" />
             <origin xyz="0.0 0.0 0.0" rpy="0 0 0" />
             <inertia ixx="0.13" ixy="0.0" ixz="0.0"
                         iyy="0.13" iyz="0.0"
                         izz="0.13" />
+        </inertial> -->
+        <inertial>
+            <mass value="720.0" />
+            <origin xyz="0.0 0.0 0.0" rpy="0 0 0" />
+            <inertia ixx="140" ixy="0.0" ixz="0.0"
+                        iyy="550" iyz="0.0"
+                        izz="550" />
         </inertial>
         <visual>
-            <origin xyz="0.0 0.0 -0.085" rpy="0 0 0" />
+            <origin xyz="0.0 0.0 0.0" rpy="0 0 0" />
+            <!-- -0.255 -->
             <geometry>
                 <!--<box size="${base_size_x} ${base_size_y} ${base_size_z}" />-->
-                <mesh filename="package://ugv_description/meshes/jasmine_ugv/jasmine_ugv.dae"/>
+                <!-- <mesh filename="package://ugv_description/meshes/jasmine_ugv/jasmine_ugv.dae" scale="3 3 3"/> -->
+                <mesh filename="package://ugv_description/meshes/lr90.dae" scale="1 1 1"/>
             </geometry>
             <material name="Grey" >
@@ -39,5 +44,5 @@
         </visual>
         <collision>
-            <origin xyz="0.0 0.0 0.0" rpy="0 0 0" />
+            <origin xyz="0 0 0" rpy="0 0 0" />
             <geometry>
                 <box size="${base_size_x} ${base_size_y} ${base_size_z}" />
@@ -48,5 +53,5 @@
         <inertial>
             <mass value="0.5" />
-            <origin xyz="0.00 0.00 0.1" rpy="0 1.5708 0" />
+            <origin xyz="0.00 0.00 0.5" rpy="0 1.5708 0" />
             <inertia ixx="0.08" ixy="0.0" ixz="0.0"
                         iyy="0.08" iyz="0.0"
@@ -54,5 +59,5 @@
         </inertial>
         <visual>
-            <origin xyz="0.00 0.00 0.1" rpy="0 0 0" />
+            <origin xyz="0.00 0.00 0.5" rpy="0 0 0" />
             <geometry>
                 <!--<box size="${base_size_x} ${base_size_y} ${base_size_z}" />-->
@@ -62,7 +67,7 @@
         </visual>
         <collision>
-            <origin xyz="0.00 0.00 0.1" rpy="0 0 0" />
+            <origin xyz="0.00 0.00 0.5" rpy="0 0 0" />
             <geometry>
-                <box size="1 1 0.01" />
+                <box size="1 1 0.02" />
             </geometry>
         </collision>
@@ -73,18 +78,16 @@
     </joint>
     <!--	Add wheels using the hlugv_wheel macro-->
-    <xacro:ugv_wheel parent="ugv_base_link" prefix="left_1" offset_x= "0.0" offset_y = "${wheel_offset_y}" offset_z = "${wheel_offset_z_from_base_link}" reflect="1" wheel_radius="${wheel_radius_big}"/>
-    <xacro:ugv_wheel parent="ugv_base_link" prefix="left_2" offset_x= "0.10550" offset_y = "${wheel_offset_y}" offset_z = "${wheel_offset_z_from_base_link}" reflect="1" wheel_radius="${wheel_radius_big}"/>
-    <xacro:ugv_wheel parent="ugv_base_link" prefix="right_1" offset_x= "0.0" offset_y = "-${wheel_offset_y}" offset_z = "${wheel_offset_z_from_base_link}" reflect="1" wheel_radius="${wheel_radius_big}"/>
-    <xacro:ugv_wheel parent="ugv_base_link" prefix="right_2" offset_x= "-0.10550" offset_y = "-${wheel_offset_y}" offset_z = "${wheel_offset_z_from_base_link}" reflect="1" wheel_radius="${wheel_radius_big}"/>
+    <xacro:ugv_wheel parent="ugv_base_link" prefix="left_1" offset_x= "-0.7" offset_y = "${wheel_offset_y}" offset_z = "${wheel_offset_z_from_base_link}"
+            reflect="1" wheel_radius="${wheel_radius}" wheel_size_y="${wheel_length}"/>
+    <xacro:ugv_wheel parent="ugv_base_link" prefix="left_2" offset_x= "0.7" offset_y = "${wheel_offset_y}" offset_z = "${wheel_offset_z_from_base_link}"
+            reflect="1" wheel_radius="${wheel_radius}" wheel_size_y="${wheel_length}"/>
+    <xacro:ugv_wheel parent="ugv_base_link" prefix="right_1" offset_x= "-0.7" offset_y = "-${wheel_offset_y}" offset_z = "${wheel_offset_z_from_base_link}"
+            reflect="1" wheel_radius="${wheel_radius}" wheel_size_y="${wheel_length}"/>
+    <xacro:ugv_wheel parent="ugv_base_link" prefix="right_2" offset_x= "0.7" offset_y = "-${wheel_offset_y}" offset_z = "${wheel_offset_z_from_base_link}"
+            reflect="1" wheel_radius="${wheel_radius}" wheel_size_y="${wheel_length}"/>
     <gazebo reference="ugv_base_link">
         <material>HLUGV/Green</material>
     </gazebo>
     <gazebo>
-        <!--
-        <plugin name="gazebo_ros_control" filename="libgazebo_ros_control.so">
-            <robotNamespace>/ugv_robot</robotNamespace>
-            <robotSimType>gazebo_ros_control/DefaultRobotHWSim</robotSimType>
-        </plugin>
-        -->
         <plugin name="differential_drive_controller" filename="libgazebo_ros_diff_drive.so">
             <alwaysOn>true</alwaysOn>
@@ -92,7 +95,7 @@
             <leftJoint>left_1_wheel_joint</leftJoint>
             <rightJoint>right_1_wheel_joint</rightJoint>
-            <wheelSeparation>0.5380</wheelSeparation>
-            <wheelDiameter>0.2410</wheelDiameter>
-            <torque>50</torque>
+            <wheelSeparation>0.96</wheelSeparation>
+            <wheelDiameter>0.52</wheelDiameter>
+            <torque>5000</torque>
             <commandTopic>/ugv/cmd_vel</commandTopic>
             <robotBaseFrame>ugv_base_link</robotBaseFrame>

File: my_ugv/ugv_description/urdf/ugv_wheel.urdf.xacro (robot description, xacro)
@@ -4,9 +4,9 @@
   <xacro:property name="M_PI" value="3.14159" />
   <!--<xacro:property name="wheel_radius" value="0.185" />-->
-  <!--<xacro:property name="wheel_size_y" value="0.0824" />-->
+  <!-- <xacro:property name="wheel_size_y" value="0.5" /> -->
   <!-- half of wheel width + half of socket width + gap -->
-  <xacro:property name="wheel_offset_z" value="-0.112" />
+  <!-- <xacro:property name="wheel_offset_z" value="-0.112" /> -->
   <!-- wheel_radius - socket height -->
-  <xacro:macro name="ugv_wheel" params="parent prefix offset_x offset_y offset_z reflect wheel_radius">
+  <xacro:macro name="ugv_wheel" params="parent prefix offset_x offset_y offset_z reflect wheel_radius wheel_size_y">
     <joint name="${prefix}_wheel_joint" type="continuous">
       <origin xyz="${offset_x } ${offset_y * reflect} ${offset_z}" rpy="0 0 0" />
@@ -14,5 +14,5 @@
       <child link="${prefix}_wheel_link" />
       <axis xyz="0 1 0" />
-      <limit effort="100" velocity="100" />
+      <limit effort="1000" velocity="1000" />
       <joint_properties damping="0.0" friction="0.0" />
       <anchor xyz="0 0 0" />
@@ -20,10 +20,19 @@
     <link name="${prefix}_wheel_link">
       <inertial>
-        <mass value="0.01" />
+        <mass value="12" />
         <origin xyz=" 0 0 0 " />
-        <inertia  ixx="0.00012411765597" ixy="0.0" ixz="0.0"
-                 iyy="0.00015218160428" iyz="0.0"
-                 izz="0.00011763977943" />
-        </inertial>
+        <!-- <inertia  ixx="0.0012411765597" ixy="0.0" ixz="0.0"
+                 iyy="0.0015218160428" iyz="0.0"
+                 izz="0.0011763977943" /> -->
+        <inertia  ixx="0.5" ixy="0.0" ixz="0.0"
+                  iyy="0.5" iyz="0.0"
+                  izz="1" />
+      </inertial>
+        <visual>
+          <origin xyz="0 0 0" rpy="${-M_PI/2} 0 0" />
+          <geometry>
+            <cylinder radius="${wheel_radius}" length="${wheel_size_y}" />
+          </geometry>
+        </visual>
         <collision>
           <origin xyz="0 0 0" rpy="${-M_PI/2} 0 0" />
@@ -41,5 +50,5 @@
         <kd>100.0</kd>
         <minDepth>0.001</minDepth>
-        <maxVel>1.0</maxVel>
+        <maxVel>100.0</maxVel>
         <!--<fdir1>1 0 0</fdir1>-->
         <!--<maxVel>1.0</maxVel>-->

Commit message: change wheel seperation

File: my_ugv/ugv_description/urdf/ugv_robot.urdf.xacro (robot description, xacro)
@@ -14,5 +14,5 @@
     <!--    <xacro:property name="wheel_offset_y" value="${(total_width - wheel_size_y) / 2}" />-->
     <!-- <xacro:property name="wheel_offset_y" value="0.48" /> -->
-    <xacro:property name="wheel_offset_x" value="0.15" />
+    <xacro:property name="wheel_offset_x" value="0.2" />
     <xacro:property name="wheel_offset_y" value="0.48" />
     <xacro:property name="wheel_offset_z_from_base_link" value="-0.72" />
@@ -43,7 +43,4 @@
                 <mesh filename="package://ugv_description/meshes/lr90.dae" scale="1 1 1"/>
             </geometry>
-            <material name="Grey" >
-                <color rgba="0.8 0.8 0.8 1"/>
-            </material>
         </visual>
         <collision>
@@ -63,10 +60,11 @@
         </inertial>
         <visual>
+            <!-- <origin xyz="-0.00 0.00 0.5" rpy="0 0 0" /> -->
             <origin xyz="-0.50 0.00 0.5" rpy="0 0 0" />
             <geometry>
                 <!--<box size="${base_size_x} ${base_size_y} ${base_size_z}" />-->
-                <!-- <mesh filename="package://ugv_description/meshes/apriltag/apriltag.dae" scale="1 1 1"/> -->
+                <mesh filename="package://ugv_description/meshes/apriltag/apriltag.dae" scale="1 1 1"/>
                 <!-- <mesh filename="package://ugv_description/meshes/emb_apriltag/emb_apriltag.dae" scale="1 1 1"/> -->
-                <mesh filename="package://ugv_description/meshes/embed_apriltag/embed_apriltag.dae" scale="1 1 1"/>
+                <!-- <mesh filename="package://ugv_description/meshes/embed_apriltag/embed_apriltag.dae" scale="1 1 1"/> -->
             </geometry>
         </visual>
@@ -99,7 +97,13 @@
     <!-- <xacro:ugv_wheel parent="ugv_base_link" prefix="rear_wheel" offset_x= "-0.7" offset_y = "0" offset_z = "${wheel_offset_z_from_base_link}"
             reflect="1" wheel_radius="${wheel_radius}" wheel_size_y="${wheel_length}"/> -->
-    <gazebo reference="ugv_base_link">
+    <!-- <gazebo reference="ugv_base_link">
         <material>HLUGV/Green</material>
-    </gazebo>
+        <material>
+            <ambient>0.19225 0.19225 0.19225 1.0</ambient>
+            <diffuse>0.50754 0.50754 0.50754 1.0</diffuse>
+            <specular>0.508273 0.508273 0.508273 1.0</specular>
+            <emissive>0.0 0.0 0.0 0.0</emissive>
+        </material>
+    </gazebo> -->
     <gazebo>
         <plugin name="differential_drive_controller" filename="libgazebo_ros_diff_drive.so">

Commit message: change to tag25h10

File: my_ugv/ugv_description/urdf/ugv_robot.urdf.xacro (robot description, xacro)
@@ -64,5 +64,6 @@
             <geometry>
                 <!--<box size="${base_size_x} ${base_size_y} ${base_size_z}" />-->
-                <mesh filename="package://ugv_description/meshes/apriltag/apriltag.dae" scale="1 1 1"/>
+                <!-- <mesh filename="package://ugv_description/meshes/apriltag/apriltag.dae" scale="1 1 1"/> -->
+                <mesh filename="package://ugv_description/meshes/tag2510/tag2510.dae" scale="1 1 1"/>
                 <!-- <mesh filename="package://ugv_description/meshes/emb_apriltag/emb_apriltag.dae" scale="1 1 1"/> -->
                 <!-- <mesh filename="package://ugv_description/meshes/embed_apriltag/embed_apriltag.dae" scale="1 1 1"/> -->

Commit message: add new combined tag

File: my_ugv/ugv_description/urdf/ugv_robot.urdf.xacro (robot description, xacro)
@@ -65,5 +65,5 @@
                 <!--<box size="${base_size_x} ${base_size_y} ${base_size_z}" />-->
                 <!-- <mesh filename="package://ugv_description/meshes/apriltag/apriltag.dae" scale="1 1 1"/> -->
-                <mesh filename="package://ugv_description/meshes/tag2510/tag2510.dae" scale="1 1 1"/>
+                <mesh filename="package://ugv_description/meshes/mix2/mix2.dae" scale="1 1 1"/>
                 <!-- <mesh filename="package://ugv_description/meshes/emb_apriltag/emb_apriltag.dae" scale="1 1 1"/> -->
                 <!-- <mesh filename="package://ugv_description/meshes/embed_apriltag/embed_apriltag.dae" scale="1 1 1"/> -->
